File: eagle/2 byte output with darlington sink/2 byte output.brd (EAGLE design)
At the start: 82.5 x 50.5 mm, 13 parts, among them IC1 74LS595N, IC2 74LS595N, X1 MKDSN1,5/8-5,08, X2 MKDSN1,5/8-5,08, X3 MKDSN1,5/5-5,08, X4 MKDSN1,5/5-5,08, X5 MKDSN1,5/2-5,08

Commit message: check in changes
Parts:
- turned C1 to 270 degrees
- turned C2 to 270 degrees
- turned IC1 to 0 degrees
- turned IC2 to 0 degrees
Connections:
- net OUT0: now also IC1.15; no longer IC1.7
- net OUT1: now also IC1.1; no longer IC1.6
- net OUT10: now also IC2.2; no longer IC2.5
- net OUT11: now also IC2.3; no longer IC2.4
- net OUT12: now also IC2.4; no longer IC2.3
- net OUT13: now also IC2.5; no longer IC2.2
- net OUT14: now also IC2.6; no longer IC2.1
- net OUT15: now also IC2.7; no longer IC2.15
- net OUT2: now also IC1.2; no longer IC1.5
- net OUT3: now also IC1.3; no longer IC1.4
- net OUT4: now also IC1.4; no longer IC1.3
- net OUT5: now also IC1.5; no longer IC1.2
- net OUT6: now also IC1.6; no longer IC1.1
- net OUT7: now also IC1.7; no longer IC1.15
- net OUT8: now also IC2.15; no longer IC2.7
- net OUT9: now also IC2.1; no longer IC2.6
Routing:
- net DP: track 45.5 -> 18.6 mm, vias 2 -> 0
- net DO: track 31.6 -> 16.2 mm
- net OUT13: track 10.5 -> 17.0 mm
- net OUT12: track 10.5 -> 17.0 mm
- net OUT11: track 10.5 -> 17.0 mm
- net OUT10: track 10.5 -> 17.0 mm
- net OUT3: track 10.5 -> 17.0 mm
- net OUT14: track 10.5 -> 17.0 mm
- net OUT1: track 10.5 -> 17.0 mm
- net OUT9: track 10.5 -> 17.0 mm
- net OUT6: track 10.5 -> 17.0 mm
- net OUT5: track 10.5 -> 17.0 mm
- net OUT4: track 10.5 -> 17.0 mm
- net OUT2: track 10.5 -> 17.0 mm
- net OUT0: track 10.5 -> 16.3 mm
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Other:
- board text added: "2 byte output with darlington array - sink 8/19"
- board text removed: "2 byte output with darlington array 7/19"
