File: eagle/2 byte output with darlington sink/2 byte output.sch (EAGLE design)
At the start: 13 parts, among them IC1 74LS595N, IC2 74LS595N, X1 MKDSN1,5/8-5,08, X2 MKDSN1,5/8-5,08, X3 MKDSN1,5/5-5,08, X4 MKDSN1,5/5-5,08, X5 MKDSN1,5/2-5,08

Commit message: periodic check in - everything working so far with breadboards.
Connections:
- net DI: now also X3-4.KL; no longer X3-2.KL
- net DO: now also X4-2.KL; no longer X4-4.KL
- net LATCH: now also X3-2.KL, X4-4.KL; no longer X3-4.KL, X4-2.KL
Changed lines of the file:
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@@
 </segment>
 <segment>
-<pinref part="X3" gate="-2" pin="KL"/>
-<wire x1="-10.16" y1="25.4" x2="-5.08" y2="25.4" width="0.1524" layer="91"/>
-<label x="-5.08" y="25.4" size="1.27" layer="95" xref="yes"/>
+<pinref part="X3" gate="-4" pin="KL"/>
+<wire x1="-10.16" y1="35.56" x2="-5.08" y2="35.56" width="0.1524" layer="91"/>
+<label x="-5.08" y="35.56" size="1.27" layer="95" xref="yes"/>
 </segment>
 </net>
@@
 </segment>
 <segment>
-<pinref part="X3" gate="-4" pin="KL"/>
-<wire x1="-10.16" y1="35.56" x2="-5.08" y2="35.56" width="0.1524" layer="91"/>
-<label x="-5.08" y="35.56" size="1.27" layer="95" xref="yes"/>
+<pinref part="X3" gate="-2" pin="KL"/>
+<wire x1="-10.16" y1="25.4" x2="-5.08" y2="25.4" width="0.1524" layer="91"/>
+<label x="-5.08" y="25.4" size="1.27" layer="95" xref="yes"/>
 </segment>
 <segment>
-<pinref part="X4" gate="-2" pin="KL"/>
-<wire x1="124.46" y1="40.64" x2="119.38" y2="40.64" width="0.1524" layer="91"/>
-<label x="119.38" y="40.64" size="1.27" layer="95" rot="MR0" xref="yes"/>
+<pinref part="X4" gate="-4" pin="KL"/>
+<wire x1="124.46" y1="30.48" x2="119.38" y2="30.48" width="0.1524" layer="91"/>
+<label x="119.38" y="30.48" size="1.27" layer="95" rot="MR0" xref="yes"/>
 </segment>
 </net>
@@
 </segment>
 <segment>
-<pinref part="X4" gate="-4" pin="KL"/>
-<wire x1="124.46" y1="30.48" x2="119.38" y2="30.48" width="0.1524" layer="91"/>
-<label x="119.38" y="30.48" size="1.27" layer="95" rot="MR0" xref="yes"/>
+<pinref part="X4" gate="-2" pin="KL"/>
+<wire x1="124.46" y1="40.64" x2="119.38" y2="40.64" width="0.1524" layer="91"/>
+<label x="119.38" y="40.64" size="1.27" layer="95" rot="MR0" xref="yes"/>
 </segment>
 </net>
