File: eagle/blockocchexdelay/blockoccdelay.brd (EAGLE design)
At the start: 91.4 x 93.7 mm, 59 parts, among them IC1 74LS14N, IC2 555, IC3 555, IC4 555, IC5 555, IC6 555, IC7 555, X1 MKDSN1,5/2-5,08, X10 MKDSN1,5/2-5,08, X11 MKDSN1,5/2-5,08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

Commit message: check in changes
Parts:
- added H4: MOUNT-HOLE3.2, holes:3,2
- added X14: MKDSN1,5/2-5,08, con-phoenix-508:MKDSN1,5/2-5,08
- moved H1 41.0 mm to (3.81, 5.97)
- moved X10 14.0 mm to (3.81, 25.4)
- moved X9 11.4 mm to (3.81, 35.6)
- moved X8 8.89 mm to (3.81, 45.7)
- moved X7 6.35 mm to (3.81, 76.2)
- moved X6 3.81 mm to (3.81, 66.0)
- moved X1 1.27 mm to (3.81, 55.9)
Connections:
- net +5V: now also X14.1
- net GND: now also X14.2
Routing:
- net TRK6: track 39.5 -> 50.1 mm
- net DCC6: track 37.9 -> 45.4 mm
- net TRK5: track 38.5 -> 45.5 mm
- net DCC1: track 40.0 -> 43.3 mm
- net TRK4: track 38.2 -> 40.6 mm
- net DCC4: track 41.0 -> 38.7 mm
- net TRK1: track 38.5 -> 40.6 mm
- net TRK2: track 38.5 -> 39.7 mm
- net DCC5: track 41.8 -> 40.8 mm
- net DCC2: track 40.0 -> 40.8 mm
- net DCC3: track 37.9 -> 38.7 mm
Other:
- board text added: "7/21/19"
- board text removed: "7/19"
