File: eagle/blockocchexdelay/blockoccdelay.sch (EAGLE design)
At the start: 59 parts, among them IC1 74LS14N, IC2 555, IC3 555, IC4 555, IC5 555, IC6 555, IC7 555, X1 MKDSN1,5/2-5,08, X10 MKDSN1,5/2-5,08, X11 MKDSN1,5/2-5,08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

Commit message: check in changes
Parts:
- added H4: MOUNT-HOLE3.2, holes:MOUNT-HOLE3.2
- added X14: MKDSN1,5/2-5,08, con-phoenix-508:MKDSN1,5/2-5,08
Connections:
- net +5V: now also X14-1.KL
- net GND: now also X14-2.KL
Other:
- moved on the sheet: H1, H2, H3, IC1P
Changed lines of the file:
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@@
 <part name="X13" library="con-phoenix-508" library_urn="urn:adsk.eagle:library:176" deviceset="MKDSN1,5/2-5,08" device="" package3d_urn="urn:adsk.eagle:package:9630/1"/>
 <part name="H3" library="holes" library_urn="urn:adsk.eagle:library:237" deviceset="MOUNT-HOLE" device="3.2" package3d_urn="urn:adsk.eagle:package:14275/1"/>
+<part name="X14" library="con-phoenix-508" library_urn="urn:adsk.eagle:library:176" deviceset="MKDSN1,5/2-5,08" device="" package3d_urn="urn:adsk.eagle:package:9630/1"/>
+<part name="GND9" library="supply1" library_urn="urn:adsk.eagle:library:371" deviceset="GND" device=""/>
+<part name="P+15" library="supply1" library_urn="urn:adsk.eagle:library:371" deviceset="+5V" device=""/>
+<part name="H4" library="holes" library_urn="urn:adsk.eagle:library:237" deviceset="MOUNT-HOLE" device="3.2" package3d_urn="urn:adsk.eagle:package:14275/1"/>
 </parts>
 <sheets>
@@
 <attribute name="VALUE" x="105.41" y="0" size="1.778" layer="96"/>
 </instance>
-<instance part="IC1" gate="P" x="172.72" y="20.32" smashed="yes">
-<attribute name="NAME" x="172.085" y="19.685" size="1.778" layer="95"/>
+<instance part="IC1" gate="P" x="208.28" y="25.4" smashed="yes">
+<attribute name="NAME" x="207.645" y="24.765" size="1.778" layer="95"/>
 </instance>
 <instance part="B1" gate="1" x="-10.16" y="71.12" smashed="yes">
@@
 <attribute name="VALUE" x="152.4" y="10.16" size="1.778" layer="96"/>
 </instance>
-<instance part="P+2" gate="1" x="172.72" y="35.56" smashed="yes">
-<attribute name="VALUE" x="170.18" y="30.48" size="1.778" layer="96" rot="R90"/>
-</instance>
-<instance part="GND2" gate="1" x="172.72" y="5.08" smashed="yes">
-<attribute name="VALUE" x="170.18" y="2.54" size="1.778" layer="96"/>
+<instance part="P+2" gate="1" x="208.28" y="40.64" smashed="yes">
+<attribute name="VALUE" x="205.74" y="35.56" size="1.778" layer="96" rot="R90"/>
+</instance>
+<instance part="GND2" gate="1" x="208.28" y="7.62" smashed="yes">
+<attribute name="VALUE" x="205.74" y="5.08" size="1.778" layer="96"/>
 </instance>
 <instance part="P+3" gate="1" x="58.42" y="91.44" smashed="yes">
@@
 <attribute name="NAME" x="135.128" y="-5.969" size="1.778" layer="95"/>
 </instance>
-<instance part="H1" gate="G$1" x="195.58" y="48.26" smashed="yes">
-<attribute name="NAME" x="197.612" y="48.8442" size="1.778" layer="95"/>
-<attribute name="VALUE" x="197.612" y="45.7962" size="1.778" layer="96"/>
-</instance>
-<instance part="H2" gate="G$1" x="195.58" y="40.64" smashed="yes">
-<attribute name="NAME" x="197.612" y="41.2242" size="1.778" layer="95"/>
-<attribute name="VALUE" x="197.612" y="38.1762" size="1.778" layer="96"/>
+<instance part="H1" gate="G$1" x="231.14" y="48.26" smashed="yes">
+<attribute name="NAME" x="233.172" y="48.8442" size="1.778" layer="95"/>
+<attribute name="VALUE" x="233.172" y="45.7962" size="1.778" layer="96"/>
+</instance>
+<instance part="H2" gate="G$1" x="231.14" y="40.64" smashed="yes">
+<attribute name="NAME" x="233.172" y="41.2242" size="1.778" layer="95"/>
+<attribute name="VALUE" x="233.172" y="38.1762" size="1.778" layer="96"/>
 </instance>
 <instance part="B2" gate="1" x="-10.16" y="121.92" smashed="yes">
@@
 <attribute name="NAME" x="53.848" y="-5.969" size="1.778" layer="95"/>
 </instance>
-<instance part="H3" gate="G$1" x="195.58" y="33.02" smashed="yes">
-<attribute name="NAME" x="197.612" y="33.6042" size="1.778" layer="95"/>
-<attribute name="VALUE" x="197.612" y="30.5562" size="1.778" layer="96"/>
+<instance part="H3" gate="G$1" x="231.14" y="33.02" smashed="yes">
+<attribute name="NAME" x="233.172" y="33.6042" size="1.778" layer="95"/>
+<attribute name="VALUE" x="233.172" y="30.5562" size="1.778" layer="96"/>
+</instance>
+<instance part="X14" gate="-1" x="180.34" y="22.86" smashed="yes">
+<attribute name="NAME" x="183.388" y="21.971" size="1.778" layer="95"/>
+</instance>
+<instance part="X14" gate="-2" x="180.34" y="17.78" smashed="yes">
+<attribute name="NAME" x="183.388" y="16.891" size="1.778" layer="95"/>
+</instance>
+<instance part="GND9" gate="1" x="175.26" y="12.7" smashed="yes">
+<attribute name="VALUE" x="172.72" y="10.16" size="1.778" layer="96"/>
+</instance>
+<instance part="P+15" gate="1" x="175.26" y="30.48" smashed="yes">
+<attribute name="VALUE" x="172.72" y="25.4" size="1.778" layer="96" rot="R90"/>
+</instance>
+<instance part="H4" gate="G$1" x="231.14" y="25.4" smashed="yes">
+<attribute name="NAME" x="233.172" y="25.9842" size="1.778" layer="95"/>
+<attribute name="VALUE" x="233.172" y="22.9362" size="1.778" layer="96"/>
 </instance>
 </instances>
@@
 <segment>
 <pinref part="IC1" gate="P" pin="VCC"/>
-<wire x1="172.72" y1="30.48" x2="172.72" y2="33.02" width="0.1524" layer="91"/>
+<wire x1="208.28" y1="35.56" x2="208.28" y2="38.1" width="0.1524" layer="91"/>
 <pinref part="P+2" gate="1" pin="+5V"/>
 </segment>
@@
 <junction x="246.38" y="96.52"/>
 </segment>
+<segment>
+<pinref part="X14" gate="-1" pin="KL"/>
+<wire x1="177.8" y1="22.86" x2="175.26" y2="22.86" width="0.1524" layer="91"/>
+<wire x1="175.26" y1="22.86" x2="175.26" y2="27.94" width="0.1524" layer="91"/>
+<pinref part="P+15" gate="1" pin="+5V"/>
+</segment>
 </net>
 <net name="GND" class="0">
@@
 <segment>
 <pinref part="IC1" gate="P" pin="GND"/>
-<wire x1="172.72" y1="10.16" x2="172.72" y2="7.62" width="0.1524" layer="91"/>
+<wire x1="208.28" y1="15.24" x2="208.28" y2="10.16" width="0.1524" layer="91"/>
 <pinref part="GND2" gate="1" pin="GND"/>
 </segment>
@@
 <junction x="243.84" y="68.58"/>
 </segment>
+<segment>
+<pinref part="X14" gate="-2" pin="KL"/>
+<wire x1="177.8" y1="17.78" x2="175.26" y2="17.78" width="0.1524" layer="91"/>
+<wire x1="175.26" y1="17.78" x2="175.26" y2="15.24" width="0.1524" layer="91"/>
+<pinref part="GND9" gate="1" pin="GND"/>
+</segment>
 </net>
