File: eagle/button debounce pos/button debounce pos.brd (EAGLE design)
At the start: 43.1 x 49 mm, 21 parts, among them IC1 74LS14N, X1 MKDSN1,5/2-5,08, X2 MKDSN1,5/6-5,08

Commit message: check in changes
Parts:
- R1, R2, R3, R4, R5, R6: value 10K -> 10k
- X1: value MKDSN1,5/2-5,08 -> MKDSN1,5/6-5,08; device con-phoenix-508:MKDSN1,5/2-5,08 -> con-phoenix-508:MKDSN1,5/6-5,08
- X2: value MKDSN1,5/6-5,08 -> MKDSN1,5/2-5,08; device con-phoenix-508:MKDSN1,5/6-5,08 -> con-phoenix-508:MKDSN1,5/2-5,08
- moved H1 52.4 mm to (5.08, 44.5)
- moved H3 52.4 mm to (5.08, 3.81)
- moved X2 35.7 mm to (3.68, 23.9), turned to 90 degrees
- moved X1 34.5 mm to (38.4, 23.7), turned to 270 degrees
- moved H2 34.3 mm to (39.4, 44.5)
- moved H4 34.3 mm to (39.4, 3.81)
- moved C1 1.27 mm to (14.0, 33.0)
- moved C3 1.27 mm to (29.2, 33.0)
- moved C4 1.27 mm to (14.0, 15.2), turned to 180 degrees
- moved C6 1.27 mm to (29.2, 15.2), turned to 180 degrees
- moved IC1 1.27 mm to (21.6, 24.1)
- moved R1 1.27 mm to (14.0, 38.1)
- moved R3 1.27 mm to (29.2, 38.1)
- moved R4 1.27 mm to (14.0, 10.2), turned to 180 degrees
- moved R6 1.27 mm to (29.2, 10.2), turned to 180 degrees
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Connections:
- net +5V: now also C1.+, C2.+, C3.+, C4.+, C5.+, C6.+, JP1.1, JP1.3, JP1.5, JP2.1, JP2.3, JP2.5, X2.1; no longer R1.2, R2.2, R3.2, R4.2, R5.2, R6.2, X1.1
- net B0: now also C1.-, R1.2; no longer C1.+, R1.1
- net B1: now also C2.-, R2.2; no longer C2.+, R2.1
- net B2: now also C3.-, R3.2; no longer C3.+, R3.1
- net B3: now also C4.-, R4.2; no longer C4.+, R4.1
- net B4: now also C5.-, R5.2; no longer C5.+, R5.1
- net B5: now also C6.-, R6.2; no longer C6.+, R6.1
- net GND: now also R1.1, R2.1, R3.1, R4.1, R5.1, R6.1, X2.2; no longer C1.-, C2.-, C3.-, C4.-, C5.-, C6.-, JP1.1, JP1.3, JP1.5, JP2.1, JP2.3, JP2.5, X1.2
- net OUT0: now also X1.1; no longer X2.1
- net OUT1: now also X1.2; no longer X2.2
- net OUT2: now also X1.3; no longer X2.3
- net OUT3: now also X1.4; no longer X2.4
- net OUT4: now also X1.5; no longer X2.5
- net OUT5: now also X1.6; no longer X2.6
Routing:
- net OUT2: track 9.44 -> 22.6 mm
- net B2: track 33.2 -> 39.0 mm
- net OUT0: track 28.6 -> 32.3 mm
- net B5: track 35.6 -> 38.9 mm
- net B1: track 26.7 -> 29.5 mm
- net B0: track 20.6 -> 23.2 mm
- net OUT1: track 16.3 -> 18.8 mm
- net OUT4: track 21.0 -> 18.5 mm
- net B3: track 20.0 -> 18.6 mm
- net OUT3: track 25.0 -> 24.3 mm
- net B4: track 28.8 -> 29.3 mm
Other:
- board size 43.1 x 49 mm -> 43.2 x 49.2 mm
- board text added: "Button De-bounce Press Low 7/19"
- board text removed: "Button Debouncer Press High 7/19"
