File: eagle/2 byte output/2 byte output.brd (EAGLE design)
At the start: 160 x 100 mm, 8 parts, among them IC1 74LS595N, IC2 74LS595N, X1 MKDSN1,5/9-5,08, X2 MKDSN1,5/8-5,08, X3 MKDSN1,5/5-5,08, X4 MKDSN1,5/5-5,08

Commit message: periodic check in - everything working so far with breadboards.
Routing:
- net LATCH: track 146.8 -> 122.6 mm
- net DI: track 47.1 -> 30.5 mm
Changed lines of the file:
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@@
 <?xml version="1.0" encoding="utf-8"?>
 <!DOCTYPE eagle SYSTEM "eagle.dtd">
-<eagle version="9.3.0">
+<eagle version="9.4.2">
 <drawing>
 <settings>
@@
 <signals>
 <signal name="DI">
-<contactref element="X3" pad="4"/>
 <contactref element="IC1" pad="14"/>
-<wire x1="5.055" y1="19.0289" x2="21.6111" y2="19.0289" width="0.4064" layer="1"/>
 <wire x1="21.6111" y1="19.0289" x2="26.67" y2="13.97" width="0.4064" layer="1"/>
 <wire x1="45.72" y1="13.97" x2="46.99" y2="12.7" width="0.4064" layer="1"/>
 <wire x1="46.99" y1="12.7" x2="46.99" y2="10.16" width="0.4064" layer="1"/>
 <wire x1="26.67" y1="13.97" x2="45.72" y2="13.97" width="0.4064" layer="1"/>
+<contactref element="X3" pad="4"/>
+<wire x1="5.055" y1="19.0289" x2="21.6111" y2="19.0289" width="0" layer="19" extent="1-1"/>
 </signal>
 <signal name="CLK">
@@
 </signal>
 <signal name="LATCH">
-<contactref element="X3" pad="2"/>
 <contactref element="X4" pad="4"/>
 <contactref element="IC1" pad="12"/>
 <contactref element="IC2" pad="12"/>
-<wire x1="5.055" y1="8.8689" x2="29.2311" y2="8.8689" width="0.4064" layer="1"/>
 <wire x1="29.2311" y1="8.8689" x2="31.75" y2="6.35" width="0.4064" layer="1"/>
 <wire x1="31.75" y1="6.35" x2="93.98" y2="6.35" width="0.4064" layer="1"/>
@@
 <wire x1="33.02" y1="12.7" x2="29.2311" y2="8.9111" width="0.4064" layer="1"/>
 <wire x1="29.2311" y1="8.9111" x2="29.2311" y2="8.8689" width="0.4064" layer="1"/>
+<contactref element="X3" pad="2"/>
+<wire x1="5.055" y1="8.8689" x2="29.2311" y2="8.9111" width="0" layer="19" extent="1-1"/>
 </signal>
 <signal name="DO">
