File: eagle/2 byte output with darlington source/2 byte output.sch (EAGLE design)
At the start: 13 parts, among them IC1 74LS595N, IC2 74LS595N, X1 MKDSN1,5/8-5,08, X2 MKDSN1,5/8-5,08, X3 MKDSN1,5/5-5,08, X4 MKDSN1,5/5-5,08, X5 MKDSN1,5/2-5,08

Commit message: check in changes
Parts:
- removed ULN1, ULN2: (no value), SparkFun-IC-Special-Function:ULN2803DIP
- added IC3, IC4: UDN2981A, uln-udn:UDN2981A
Connections:
- removed net COM: ULN1.10, ULN2.10, X5-1.KL
- removed net OUT0: IC1A.QH, ULN1.1
- removed net OUT1: IC1A.QG, ULN1.2
- removed net OUT10: IC2A.QF, ULN2.3
- removed net OUT11: IC2A.QE, ULN2.4
- removed net OUT12: IC2A.QD, ULN2.5
- removed net OUT13: IC2A.QC, ULN2.6
- removed net OUT14: IC2A.QB, ULN2.7
- removed net OUT15: IC2A.QA, ULN2.8
- removed net OUT2: IC1A.QF, ULN1.3
- removed net OUT3: IC1A.QE, ULN1.4
- removed net OUT4: IC1A.QD, ULN1.5
- removed net OUT5: IC1A.QC, ULN1.6
- removed net OUT6: IC1A.QB, ULN1.7
- removed net OUT7: IC1A.QA, ULN1.8
- removed net OUT8: IC2A.QH, ULN2.1
- removed net OUT9: IC2A.QG, ULN2.2
- new net N$17: IC1A.QA, IC3.I1
- new net N$18: IC1A.QB, IC3.I2
- new net N$19: IC1A.QC, IC3.I3
- new net N$20: IC1A.QD, IC3.I4
- new net N$21: IC1A.QE, IC3.I5
- new net N$22: IC1A.QF, IC3.I6
- new net N$23: IC1A.QG, IC3.I7
- new net N$24: IC1A.QH, IC3.I8
- new net N$25: IC2A.QA, IC4.I1
- new net N$26: IC2A.QB, IC4.I2
- new net N$27: IC2A.QC, IC4.I3
- new net N$28: IC2A.QD, IC4.I4
- new net N$29: IC2A.QE, IC4.I5
- new net N$30: IC2A.QF, IC4.I6
- new net N$31: IC2A.QG, IC4.I7
- new net N$32: IC2A.QH, IC4.I8
- new net VS: IC3.VS, IC4.VS, X5-1.KL
- net GND: now also IC3.GND, IC4.GND; no longer ULN1.9, ULN2.9
- net N$1: now also IC3.O4, X1-4.KL; no longer ULN1.18, X1-1.KL
- net N$10: now also IC4.O3, X2-3.KL; no longer ULN2.17, X2-2.KL
- net N$11: now also IC4.O2, X2-2.KL; no longer ULN2.16, X2-3.KL
- net N$12: now also IC4.O1, X2-1.KL; no longer ULN2.15, X2-4.KL
- net N$13: now also IC4.O5; no longer ULN2.14
- net N$14: now also IC4.O6; no longer ULN2.13
- net N$15: now also IC4.O7; no longer ULN2.12
- net N$16: now also IC4.O8; no longer ULN2.11
- net N$2: now also IC3.O3, X1-3.KL; no longer ULN1.17, X1-2.KL
- net N$3: now also IC3.O2, X1-2.KL; no longer ULN1.16, X1-3.KL
- net N$4: now also IC3.O1, X1-1.KL; no longer ULN1.15, X1-4.KL
- net N$5: now also IC3.O5; no longer ULN1.14
- net N$6: now also IC3.O7, X1-7.KL; no longer ULN1.13, X1-6.KL
- net N$7: now also IC3.O8, X1-8.KL; no longer ULN1.12, X1-7.KL
- net N$8: now also IC3.O6, X1-6.KL; no longer ULN1.11, X1-8.KL
- net N$9: now also IC4.O4, X2-4.KL; no longer ULN2.18, X2-1.KL
Other:
- moved on the sheet: X1-1, X1-2, X1-3, X1-4, X1-5, X1-6, X1-7, X1-8, X2-1, X2-2, X2-3, X2-4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

Commit message: periodic check in - everything working so far with breadboards.
Connections:
- net DI: now also X3-4.KL; no longer X3-2.KL
- net DO: now also X4-2.KL; no longer X4-4.KL
- net LATCH: now also X3-2.KL, X4-4.KL; no longer X3-4.KL, X4-2.KL
Changed lines of the file:
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@@
 </segment>
 <segment>
-<pinref part="X3" gate="-2" pin="KL"/>
-<wire x1="-10.16" y1="25.4" x2="-5.08" y2="25.4" width="0.1524" layer="91"/>
-<label x="-5.08" y="25.4" size="1.27" layer="95" xref="yes"/>
+<pinref part="X3" gate="-4" pin="KL"/>
+<wire x1="-10.16" y1="35.56" x2="-5.08" y2="35.56" width="0.1524" layer="91"/>
+<label x="-5.08" y="35.56" size="1.27" layer="95" xref="yes"/>
 </segment>
 </net>
@@
 </segment>
 <segment>
-<pinref part="X3" gate="-4" pin="KL"/>
-<wire x1="-10.16" y1="35.56" x2="-5.08" y2="35.56" width="0.1524" layer="91"/>
-<label x="-5.08" y="35.56" size="1.27" layer="95" xref="yes"/>
+<pinref part="X3" gate="-2" pin="KL"/>
+<wire x1="-10.16" y1="25.4" x2="-5.08" y2="25.4" width="0.1524" layer="91"/>
+<label x="-5.08" y="25.4" size="1.27" layer="95" xref="yes"/>
 </segment>
 <segment>
-<pinref part="X4" gate="-2" pin="KL"/>
-<wire x1="124.46" y1="40.64" x2="119.38" y2="40.64" width="0.1524" layer="91"/>
-<label x="119.38" y="40.64" size="1.27" layer="95" rot="MR0" xref="yes"/>
+<pinref part="X4" gate="-4" pin="KL"/>
+<wire x1="124.46" y1="30.48" x2="119.38" y2="30.48" width="0.1524" layer="91"/>
+<label x="119.38" y="30.48" size="1.27" layer="95" rot="MR0" xref="yes"/>
 </segment>
 </net>
@@
 </segment>
 <segment>
-<pinref part="X4" gate="-4" pin="KL"/>
-<wire x1="124.46" y1="30.48" x2="119.38" y2="30.48" width="0.1524" layer="91"/>
-<label x="119.38" y="30.48" size="1.27" layer="95" rot="MR0" xref="yes"/>
+<pinref part="X4" gate="-2" pin="KL"/>
+<wire x1="124.46" y1="40.64" x2="119.38" y2="40.64" width="0.1524" layer="91"/>
+<label x="119.38" y="40.64" size="1.27" layer="95" rot="MR0" xref="yes"/>
 </segment>
 </net>

Commit message: periodic check-in
Parts:
- removed X3, X4: MKDSN1,5/5-5,08, con-phoenix-508:MKDSN1,5/5-5,08
- added JP1, JP2: (no value), pinhead:PINHD-1X5/90
- IC3, IC4: value UDN2981A -> MIC2981A
Connections:
- net CLK: now also JP1.3, JP2.3; no longer X3-3.KL, X4-3.KL
- net DI: now also JP1.4; no longer X3-4.KL
- net DO: now also JP2.2; no longer X4-2.KL
- net GND: now also JP1.1, JP2.5; no longer X3-1.KL, X4-5.KL
- net LATCH: now also JP1.2, JP2.4; no longer X3-2.KL, X4-4.KL
- net VCC: now also JP1.5, JP2.1; no longer X3-5.KL, X4-1.KL
