File: eagle/2 byte input/2 byte input.brd (EAGLE design)
At the start: 85.1 x 44.1 mm, 26 parts, among them IC1 74LS165N, IC2 74LS165N, X3 MKDSN1,5/8-5,08, X5 MKDSN1,5/8-5,08

Commit message: added pdf file of schematics and boards, removed button debounce and servo driver
Parts:
- R1: value (none) -> 4.7k
Changed lines of the file:
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@@
 <?xml version="1.0" encoding="utf-8"?>
 <!DOCTYPE eagle SYSTEM "eagle.dtd">
-<eagle version="9.4.2">
+<eagle version="9.5.0">
 <drawing>
 <settings>
@@
 <attribute name="VALUE" x="52.197" y="18.415" size="1.27" layer="27" ratio="10"/>
 </element>
-<element name="R1" library="resistor" library_urn="urn:adsk.eagle:library:348" package="0207/2V" package3d_urn="urn:adsk.eagle:package:23490/1" value="" x="5.08" y="33.02" smashed="yes" rot="R90">
-<attribute name="VALUE" x="7.3152" y="32.9692" size="1.27" layer="27" ratio="10" rot="R90"/>
-</element>
+<element name="R1" library="resistor" library_urn="urn:adsk.eagle:library:348" package="0207/2V" package3d_urn="urn:adsk.eagle:package:23490/1" value="4.7k" x="5.08" y="33.02" smashed="yes" rot="R90"/>
 <element name="R10" library="resistor" library_urn="urn:adsk.eagle:library:348" package="0207/2V" package3d_urn="urn:adsk.eagle:package:23490/1" value="" x="50.8" y="33.02" smashed="yes" rot="R90">
 <attribute name="VALUE" x="53.0352" y="32.9692" size="1.27" layer="27" ratio="10" rot="R90"/>
