File: eagle/blockocctwodelay/blockoccdelay.sch (EAGLE design)
At the start: 58 parts, among them IC1 74LS14N, IC2 555, IC3 555, IC4 555, IC5 555, IC6 555, IC7 555, X1 MKDSN1,5/2-5,08, X10 MKDSN1,5/2-5,08, X11 MKDSN1,5/2-5,08, X12 MKDSN1,5/2-5,08, X13 MKDSN1,5/2-5,08, X14 MKDSN1,5/2-5,08, X2 MKDSN1,5/2-5,08, X3 MKDSN1,5/2-5,08, X4 MKDSN1,5/2-5,08, X5 MKDSN1,5/2-5,08, X6 MKDSN1,5/2-5,08, X7 MKDSN1,5/2-5,08, X8 MKDSN1,5/2-5,08, X9 MKDSN1,5/2-5,08

Commit message: periodic checkin
Parts:
- removed B1, B4, B5, B6: (no value), rectifier:GBU4
- removed C1, C11, C7, C9: 10uf, resistor:CPOL-USE2.5-6
- removed C10, C12, C3, C8: 0.01uf, resistor:C-EU050-035X075
- removed IC2, IC5, IC6, IC7: 555, SparkFun-IC-Special-Function:555P
- removed OK8, OK9: LTV826, optocoupler:LTV826
- removed R1, R11, R7, R9: 33r, resistor:R-EU_0207/2V
- removed R10, R12, R2, R8: 120k, resistor:R-US_0309/V
- removed X1, X10, X12, X13, X4, X5, X8, X9: MKDSN1,5/2-5,08, con-phoenix-508:MKDSN1,5/2-5,08
Connections:
- removed net DCC3: B1.AC1, R1.1, X1-1.KL
- removed net DCC4: B4.AC1, R7.1, X8-1.KL
- removed net DCC5: B5.AC1, R9.1, X9-1.KL
- removed net DCC6: B6.AC1, R11.1, X10-1.KL
- removed net N$1: B1.+, B1.-
- removed net N$16: B5.+, B5.-
- removed net N$17: OK9A.A, R9.2
- removed net N$18: C10.1, IC6.CON
- removed net N$19: B6.+, B6.-
- removed net N$2: OK8A.A, R1.2
- removed net N$20: OK9B.A, R11.2
- removed net N$21: C12.1, IC7.CON
- removed net N$23: IC1E.O, X12-1.KL
- removed net N$24: IC1F.O, X13-1.KL
- removed net N$3: C3.1, IC2.CON
- removed net N$5: B4.+, B4.-
- removed net N$6: OK8B.A, R7.2
- removed net N$7: IC1B.O, X4-1.KL
- removed net N$8: C8.1, IC5.CON
- removed net N$9: IC1C.O, X5-1.KL
- removed net RAW3: IC1E.I, IC2.OUT, X12-2.KL
- removed net RAW4: IC1B.I, IC5.OUT, X4-2.KL
- removed net RAW5: IC1F.I, IC6.OUT, X13-2.KL
- removed net RAW6: IC1C.I, IC7.OUT, X5-2.KL
- removed net TRI: C1.+, IC2.TRE, IC2.TRI, OK8A.COL, R2.1
- removed net TRI3: C7.+, IC5.TRE, IC5.TRI, OK8B.COL, R8.1
- removed net TRI4: C9.+, IC6.TRE, IC6.TRI, OK9A.COL, R10.1
- removed net TRI5: C11.+, IC7.TRE, IC7.TRI, OK9B.COL, R12.1
- removed net TRK3: B1.AC2, OK8A.C, X1-2.KL
- removed net TRK4: B4.AC2, OK8B.C, X8-2.KL
- removed net TRK5: B5.AC2, OK9A.C, X9-2.KL
- removed net TRK6: B6.AC2, OK9B.C, X10-2.KL
- net +5V: no longer IC2./RES, IC2.VCC+, IC5./RES, IC5.VCC+, IC6./RES, IC6.VCC+, IC7./RES, IC7.VCC+, R10.2, R12.2, R2.2, R8.2
- net GND: no longer C1.-, C10.2, C11.-, C12.2, C3.2, C7.-, C8.2, C9.-, IC2.GND, IC5.GND, IC6.GND, IC7.GND, OK8A.EMIT, OK8B.EMIT, OK9A.EMIT, OK9B.EMIT

Commit message: periodic check in
Other:
- moved on the sheet: H1, H2, H3, H4, IC1A, IC1D, IC1P, X11-1, X11-2, X14-1, X14-2, X2-1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
