File: eagle/IR Sensor/IR Sensor.sch (EAGLE design)
At the start: 14 parts, among them IC1 LM393N

Commit message: periodic check in
Parts:
- removed LED3: (no value), led:LED5MM
- removed Q1: (no value), SparkFun-Sensors:LTR-301
- added SENS-1: TCRT5000, qfm-trx1-24g:TCRT5000
- C1, C2: device resistor:C-EU025_050-055X075 -> resistor:C-US050-045X075
Connections:
- removed net N$4: Q1.C, R3.1
- net GND: now also SENS-1.P$2, SENS-1.P$4; no longer LED3.C, Q1.E
- net N$3: now also SENS-1.P$3; no longer LED3.A
- net N$5: now also R3.1, SENS-1.P$1
Other:
- moved on the sheet: C2, IC1A, JP1, LED2, R2, R4, R5, R6
