File: eagle/node/node.sch (EAGLE design)
At the start: 19 parts, among them IC2 7805TV, X1 MKDSN1,5/2-5,08, X2 MKDSN1,5/2-5,08, X3 MKDSN1,5/2-5,08, X4 MKDSN1,5/2-5,08, X5 MKDSN1,5/3-5,08, X6 MKDSN1,5/3-5,08

Commit message: periodic check in - everything working so far with breadboards.
Parts:
- removed X5, X6: MKDSN1,5/3-5,08, con-phoenix-508:MKDSN1,5/3-5,08
- added H3, H4: MOUNT-HOLE3.2, holes:MOUNT-HOLE3.2
- added JP2, JP6: (no value), pinhead:PINHD-1X6
- added JP3: (no value), pinhead:PINHD-1X5
- added JP4, JP5: (no value), pinhead:PINHD-1X2
Connections:
- new net ICE: JP2.3, U$1.D11
- new net LB1: JP6.4, U$1.D3
- new net LB2: JP6.5, U$1.D4
- new net LCLOCK: JP6.2, U$1.A5
- new net LDATA: JP6.3, U$1.A4
- new net N$10: JP5.2, U$3.DI
- new net N$11: JP4.1, U$3.RO
- net DI: now also JP5.1; no longer U$3.DI
- net GND: now also JP2.6, JP3.5, JP6.6
- net ICLOCK: now also JP2.4, U$1.D9; no longer U$1.D13, X5-2.KL
- net IDATA: now also JP2.2, U$1.D12; no longer U$1.D9, X5-3.KL
- net ILATCH: now also JP2.5, U$1.D8; no longer U$1.D10, X5-1.KL
- net OCLOCK: now also JP3.3, U$1.D6; no longer U$1.D12, X6-2.KL
- net ODATA: now also JP3.2, U$1.D7; no longer U$1.D11, X6-3.KL
- net OLATCH: now also JP3.4, U$1.D5; no longer U$1.D8, X6-1.KL
- net RO: now also JP4.2; no longer U$3.RO
- net VCC: now also JP2.1, JP3.1, JP6.1
Other:
- note added: "LCD Connector"
- note added: "output 12v from power supply??"
- moved on the sheet: H1, H2

Commit message: periodic check-in
Parts:
- added JP7: (no value), pinhead:PINHD-1X4/90
- JP2: device pinhead:PINHD-1X6 -> pinhead:PINHD-1X6/90
- JP3: device pinhead:PINHD-1X5 -> pinhead:PINHD-1X5/90
Connections:
- removed net LCLOCK: JP6.2, U$1.A5
- removed net LDATA: JP6.3, U$1.A4
- new net SCL: JP6.2, JP7.2, U$1.A5
- new net SDA: JP6.3, JP7.3, U$1.A4
- net GND: now also JP7.1, X1-2.KL; no longer X1-1.KL
- net N$2: now also X1-1.KL; no longer X1-2.KL
- net VCC: now also JP7.4
Other:
- note added: "Servo Driver"
- moved on the sheet: JP6, X1-1, X1-2

Commit message: added pdf file of schematics and boards, removed button debounce and servo driver
Other:
- note removed: "output 12v from power supply??"
Changed lines of the file:
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@@
 <text x="137.16" y="55.88" size="2.54" layer="91">Bit Output</text>
 <text x="91.44" y="76.2" size="2.54" layer="91">RS485 Interface</text>
-<text x="-22.86" y="99.06" size="2.54" layer="91">output 12v from power supply??</text>
 <text x="200.66" y="55.88" size="2.54" layer="91">LCD Connector</text>
 <text x="175.26" y="55.88" size="2.54" layer="91">Servo Driver</text>

Commit message: periodic checkin
Parts:
- removed C10, C8, C9: 0.1uf, resistor:C-EU025-025X050
- removed C3: 100/25, resistor:CPOL-USE2.5-7
- removed C4: 10uf/25v, resistor:CPOL-USE2-4
- removed D1: 1N4002, diode:1N4004
- removed IC2: 7805TV, linear:7805TV
- removed JP1: (no value), pinhead:PINHD-1X2
- removed JP6: (no value), pinhead:PINHD-1X6
- removed R1: 120R, resistor:R-US_0207/2V
- removed U$1: PRO-MINI-2, Arduino-clone:PRO-MINI-2
- removed U$3: MAX485DIL, SparkFun-DigitalIC:MAX485DIL
- removed X2, X3, X4: MKDSN1,5/2-5,08, con-phoenix-508:MKDSN1,5/2-5,08
- added M1: ARDUINO-NANO-3.0, diy-modules:ARDUINO-NANO-3.0
- JP4: device pinhead:PINHD-1X2 -> pinhead:PINHD-1X7
- JP5: device pinhead:PINHD-1X2 -> pinhead:PINHD-1X6
Connections:
- removed net A: R1.1, U$3.A, X2-1.KL, X3-1.KL
- removed net B: JP1.2, U$3.B, X2-2.KL, X3-2.KL
- removed net DE: U$1.D2, U$3.DE, U$3.RE
- removed net LB1: JP6.4, U$1.D3
- removed net LB2: JP6.5, U$1.D4
- removed net N$1: C3.+, C8.1, D1.C, IC2.VI
- removed net N$10: JP5.2, U$3.DI
- removed net N$11: JP4.1, U$3.RO
- removed net N$2: D1.A, X1-1.KL
- removed net N$3: JP1.1, R1.2
- new net AI0: JP5.1, M1.A0
- new net AI1: JP5.2, M1.A1
- new net AI2: JP5.3, M1.A2
- new net AI3: JP5.4, M1.A3
- new net DI0: JP4.1, M1.D2
- new net DI1: JP4.2, M1.D3
- new net DI2: JP4.3, M1.D4
- new net DI3: JP4.4, M1.D10
- new net DI4: JP4.5, M1.D13/SCK
- net DI: now also M1.D0/TXD; no longer JP5.1, U$1.TX0
- net GND: now also JP4.7, JP5.6, M1.GND.1, M1.GND.2; no longer C10.2, C3.-, C4.-, C8.2, C9.2, IC2.GND, JP6.6, U$1.GND, U$1.GND2, U$3.GND, X4-2.KL
- net ICE: now also M1.D11/MOSI; no longer U$1.D11
- net ICLOCK: now also M1.D9; no longer U$1.D9
- net IDATA: now also M1.D12/MISO; no longer U$1.D12
- net ILATCH: now also M1.D8; no longer U$1.D8
- net OCLOCK: now also M1.D6; no longer U$1.D6
- net ODATA: now also M1.D7; no longer U$1.D7
- net OLATCH: now also M1.D5; no longer U$1.D5
- net RO: now also M1.D1/RXD; no longer JP4.2, U$1.RX1
- net SCL: now also M1.A5; no longer JP6.2, U$1.A5
- net SDA: now also M1.A4; no longer JP6.3, U$1.A4
- net VCC: now also JP4.6, JP5.5, M1.AREF, M1.VIN, X1-1.KL; no longer C10.1, C4.+, C9.1, IC2.VO, JP6.1, U$1.VCC, U$3.VCC, X4-1.KL
Other:
- note added: "Arduino Nano"
- note removed: "Arduino Pro Mini"
- note removed: "LCD Connector"
- note removed: "Power"
- note removed: "RS485 Interface"
- moved on the sheet: H1, H2, H3, H4, JP2, JP3, JP7

Commit message: periodic check in
Parts:
- removed JP4: (no value), pinhead:PINHD-1X7
- added JP1: (no value), pinhead:PINHD-1X4/90
- added JP10, JP11: RJ45, SparkFun-Connectors:RJ45-8PTH
- added JP12: (no value), pinhead:PINHD-1X6
- added JP6, JP8, JP9: (no value), pinhead:PINHD-1X2
- added R2: 120R, resistor:R-US_0207/2V
- added U$1: MAX485, SparkFun-DigitalIC:MAX485DIL
Connections:
- removed net DI0: JP4.1, M1.D2
- removed net DI1: JP4.2, M1.D3
- removed net DI2: JP4.3, M1.D4
- removed net DI3: JP4.4, M1.D10
- removed net DI4: JP4.5, M1.D13/SCK
- new net A: JP10.4, JP11.4, JP9.1, U$1.A
- new net B: JP10.5, JP11.5, R2.1, U$1.B
- new net D10: JP12.3, M1.D10
- new net D13: JP12.4, M1.D13/SCK
- new net D3: JP12.1, M1.D3
- new net D4: JP12.2, M1.D4
- new net DE: M1.D2, U$1.DE, U$1.RE
- new net N$1: JP9.2, R2.2
- new net N$10: JP8.1, U$1.DI
- new net N$6: JP6.2, U$1.RO
- net DI: now also JP8.2
- net GND: now also JP1.4, JP10.1, JP10.2, JP11.1, JP11.2, JP12.6, U$1.GND; no longer JP4.7
- net RO: now also JP6.1
- net SCL: now also JP1.3
- net SDA: now also JP1.2
- net VCC: now also JP1.1, JP12.5, U$1.VCC; no longer JP4.6
Other:
- note added: "LCD"
- moved on the sheet: H1, H2, H3, H4
