File: kicad/1 byte input/1 byte input.kicad_pcb (KiCad board)
At the start: 2 copper layers, 59.7 x 47 mm, 8 parts, among them J1 Conn_01x06, J2 Conn_01x06, J3 Conn_01x08, U1 74LS165

Commit message: periodic check in
Parts:
- moved C1 2.54 mm to (72.4, 76.2), turned to 270 degrees
Routing:
- net +5V: track 0.00 -> 92.3 mm
- net GND: track 0.00 -> 78.3 mm, vias 0 -> 2
- net SO: track 38.4 -> 45.1 mm
- net IN5: track 34.3 -> 30.5 mm
- net IN1: track 37.8 -> 40.6 mm, vias 1 -> 0
- net IN3: track 22.6 -> 20.3 mm
- net IN6: track 34.9 -> 33.0 mm
- net IN2: track 29.7 -> 31.5 mm
- net SI: track 26.2 -> 27.9 mm
- net IN4: track 16.3 -> 17.8 mm
- net CE: track 60.8 -> 61.6 mm, vias 0 -> 1
- net IN7: track 36.2 -> 35.6 mm
- net IN8: track 37.5 -> 38.1 mm
- net LATCH: vias 0 -> 1
- removed copper zone on F.Cu, net +5V
- removed copper zone on B.Cu, net GND

Commit message: added dcc sniffer, conversion to kicad 6
Other:
- net class Default removed
