File: kicad/2 byte input/2 byte input.kicad_pcb (KiCad board)
At the start: 2 copper layers, 100.6 x 47 mm, 12 parts, among them J1 Conn_01x06, J2 Conn_01x06, J3 Conn_01x08, J4 Conn_01x08, U1 74LS165, U2 74LS165

Commit message: periodic check in
Parts:
- moved C2 2.62 mm to (120.7, 76.2), turned to 270 degrees
- moved C1 2.54 mm to (72.5, 76.2), turned to 270 degrees
Routing:
- net +5V: track 0.00 -> 162.6 mm
- net GND: track 0.00 -> 151.8 mm, vias 0 -> 4
- net SI: track 52.5 -> 75.6 mm, vias 0 -> 3
- net SO: track 38.4 -> 45.1 mm
- net IN5B: track 32.9 -> 27.9 mm
- net IN1: track 37.8 -> 41.7 mm, vias 1 -> 0
- net IN5: track 34.3 -> 30.5 mm
- net SX: track 17.2 -> 21.0 mm, vias 0 -> 1
- net IN2B: track 30.8 -> 34.0 mm
- net IN6B: track 33.1 -> 30.5 mm
- net IN3: track 22.6 -> 20.3 mm
- net IN8B: track 33.3 -> 35.6 mm
- net IN1B: track 42.6 -> 44.4 mm, vias 1 -> 0
- net IN6: track 34.9 -> 33.0 mm
- net IN2: track 29.7 -> 31.5 mm
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- removed copper zone on F.Cu, net +5V
- removed copper zone on B.Cu, net GND

Commit message: added dcc sniffer, conversion to kicad 6
Other:
- net class Default removed
