File: kicad/2 byte output mirrored/2 byte output mirrored.kicad_pcb (KiCad board)
At the start: 2 copper layers, 98.5 x 51.3 mm, 12 parts, among them J1 Conn_01x05_Male, J2 Conn_01x05_Female, J3 Screw_Terminal_01x16, J4 Screw_Terminal_01x02, U1 74HCT595, U2 ULN2803A, U3 74HCT595, U4 ULN2803A

Commit message: added dcc sniffer, conversion to kicad 6
Other:
- net class Default removed
