File: kicad/hexblockocc/hexblockocc.kicad_pcb (KiCad board)
At the start: 2 copper layers, 99.7 x 92.7 mm, 51 parts, among them J101 Conn_01x02, J102 Conn_01x02, J103 Conn_01x12, J104 Conn_01x12, U101 74LS14, U201 LTV8141, U202 NE555, U301 LTV8141, U302 NE555, U401 LTV8141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

Commit message: periodic check in
Routing:
- net +5V: track 0.00 -> 291.3 mm
- net /detection f/OUT: track 79.1 -> 86.1 mm
- net /detection e/OUT: track 64.5 -> 70.7 mm
- net /detection d/OUT: track 47.5 -> 52.7 mm
- net /detection c/OUT: track 43.9 -> 48.8 mm, vias 0 -> 1
- net Net-(C701-Pad1): track 26.4 -> 27.9 mm
- net Net-(C301-Pad1): track 26.4 -> 27.9 mm
- net Net-(C601-Pad1): track 26.4 -> 27.9 mm
- net Net-(C501-Pad1): track 26.4 -> 27.9 mm
- net Net-(C401-Pad1): track 26.4 -> 27.9 mm
- net Net-(C201-Pad1): track 26.4 -> 27.8 mm
- removed copper zone on F.Cu, net +5V

Commit message: added dcc sniffer, conversion to kicad 6
Other:
- net class Default removed
