File: kicad/node/node.kicad_pcb (KiCad board)
At the start: 2 copper layers, 15 parts, among them J1 Power, J10 Digital Pins, J11 RJ45, J12 RJ45, J13 Decouple, J14 Decouple, J2 Input, J3 Output, J4 LCD, J6 Termination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

Commit message: check in
Parts:
- removed J13, J14: Decouple, Connector_PinHeader_2.54mm:PinHeader_1x02_P2.54mm_Vertical
- added  : , MountingHole:MountingHole_3.2mm_M3, F.Cu at (67.8, 48.8)
- added  : , MountingHole:MountingHole_3.2mm_M3, F.Cu at (67.8, 117.6)
- added  : , MountingHole:MountingHole_3.2mm_M3, F.Cu at (128.8, 117.6)
- added  : , MountingHole:MountingHole_3.2mm_M3, F.Cu at (128.8, 48.8)
- added J20: , Connector_PinHeader_2.54mm:PinHeader_1x04_P2.54mm_Vertical, F.Cu at (99.1, 92.1)
- moved J10 29.1 mm to (66.5, 91.4), turned to 180 degrees
- moved R1 25.7 mm to (113.0, 101.0), turned to 0 degrees
- moved J9 23.2 mm to (66.5, 59.9)
- moved J6 16.6 mm to (106.2, 101.1), turned to 90 degrees
- moved J1 15.3 mm to (114.3, 49.5), turned to 180 degrees
- moved J8 12.5 mm to (128.5, 103.6)
- moved J4 12.4 mm to (68.8, 106.9)
- moved J12 12.4 mm to (99.6, 107.7)
- moved A1 11.0 mm to (93.2, 86.9)
- moved J11 10.1 mm to (79.2, 107.7)
- moved U2 9.43 mm to (103.6, 84.3), turned to 0 degrees
- moved J2 0.36 mm to (128.5, 67.1)
- moved J3 0.36 mm to (128.5, 86.6)
Connections:
- A1 pad 17: Net-(A1-Pad17) -> (no net)
- A1 pad 25: Net-(A1-Pad25) -> (no net)
- A1 pad 26: Net-(A1-Pad26) -> (no net)
- A1 pad 27: Net-(A1-Pad27) -> (no net)
- A1 pad 28: Net-(A1-Pad28) -> (no net)
- A1 pad 3: Net-(A1-Pad3) -> (no net)
- J11 pad 3: Net-(J11-Pad3) -> (no net)
- J11 pad 6: Net-(J11-Pad6) -> (no net)
- J11 pad 7: Net-(J11-Pad7) -> (no net)
- J11 pad 8: Net-(J11-Pad8) -> (no net)
- J12 pad 3: Net-(J12-Pad3) -> (no net)
- J12 pad 6: Net-(J12-Pad6) -> (no net)
- J12 pad 7: Net-(J12-Pad7) -> (no net)
- J12 pad 8: Net-(J12-Pad8) -> (no net)
Routing:
- net SDA: track 0.00 -> 118.0 mm
- net SCL: track 0.00 -> 111.7 mm
- net B: track 0.00 -> 60.1 mm
- net A: track 0.00 -> 51.8 mm
- net D10: track 0.00 -> 49.8 mm
- net OLATCH: track 0.00 -> 45.7 mm
- net ODATA: track 0.00 -> 45.7 mm
- net OCLOCK: track 0.00 -> 45.7 mm
- net D13: track 0.00 -> 43.6 mm
- net IDATA: track 0.00 -> 42.9 mm
- net ICE: track 0.00 -> 42.9 mm
- net ICLOCK: track 0.00 -> 41.8 mm
- net ILATCH: track 0.00 -> 41.8 mm
- net D4: track 0.00 -> 37.5 mm
- net D3: track 0.00 -> 37.2 mm
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- added copper zone on F.Cu, net VCC
Other:
- board outline added: 69.2 x 77.5 mm
- board text added: "+5V"
- board text added: "A0"
- board text added: "A1"
- board text added: "A2"
- board text added: "A3"
- board text added: "CE"
- board text added: "CLK"
- board text added: "CLOCK"
- board text added: "D10"
- board text added: "D13"
- board text added: "D4"
- board text added: "D5"
- board text added: "DATA"
- board text added: "GND"
- board text added: "INPUT"
- board text added: "LATCH"
- board text added: "LCD"
- board text added: "NODE 9/7/20"
- board text added: "OUTPUT"
- board text added: "SERVO"
- board text added: "VCC"
- board text added: "decouple"
- board text added: "termination"

Commit message: periodic check in
Routing:
- net VCC: track 0.00 -> 276.4 mm
- net SDA: track 118.0 -> 132.6 mm
- net SCL: track 111.7 -> 124.7 mm
- removed copper zone on F.Cu, net VCC
Other:
- board text added: "NODE 3/28/21"
- board text removed: "NODE 9/7/20"

Commit message: added dcc sniffer, conversion to kicad 6
Other:
- net class Default removed
- net class Power removed
