File: kicad/pihat485/pihat485.kicad_pcb (KiCad board)
At the start: 2 copper layers, 38.1 x 45.1 mm, 6 parts, among them J1 Conn_02x07_Odd_Even, J2 Conn_01x02, J3 RJ45, J4 RJ45, U1 MAX485E

Commit message: added dcc sniffer, conversion to kicad 6
Other:
- net class Default removed
