File: kicad/quadrelay/quadrelay.kicad_pcb (KiCad board)
At the start: 2 copper layers, 88.9 x 58.4 mm, 25 parts, among them J1 Conn_01x03, J2 Conn_01x03, J3 Conn_01x03, J4 Conn_01x03, J5 Conn_01x06, K1 G5LE-1, K2 G5LE-1, K3 G5LE-1, K4 G5LE-1

Commit message: periodic check in
Routing:
- net G1: track 38.9 -> 44.6 mm
- net G3: track 28.2 -> 33.5 mm
- net +5V: track 142.4 -> 147.6 mm
- net G4: track 42.9 -> 47.4 mm
- net G2: track 27.0 -> 30.7 mm

Commit message: added dcc sniffer, conversion to kicad 6
Other:
- net class Default removed
