File: kicad/single led blinker/single led blinker.kicad_pcb (KiCad board)
At the start: 2 copper layers, 45.5 x 49.8 mm, 18 parts, among them J1 Conn_01x02, J2 Conn_01x02, J3 Conn_01x02, J4 Conn_01x02, J5 Conn_01x02, Q1 NDP6020P, Q2 NDP6020P, U1 NE555P

Commit message: periodic check in
Parts:
- moved U1 1.27 mm to (119.4, 85.3)
- moved D1 1.27 mm to (127.3, 100.3)
- moved R1 1.27 mm to (128.3, 81.5)
- moved R3 1.27 mm to (118.1, 96.8)
- moved C1 1.02 mm to (123.2, 72.4)
Routing:
- net +5V: track 0.00 -> 102.8 mm
- net GBLINK: track 33.0 -> 41.7 mm
- net Net-(C1-Pad1): track 28.7 -> 34.5 mm
- net GSOLID: track 37.7 -> 42.9 mm
- net Net-(Q1-Pad2): track 24.4 -> 27.7 mm
- net LEDA: track 11.7 -> 13.5 mm
- net Net-(D1-Pad1): track 14.2 -> 15.5 mm
- net Net-(R1-Pad1): track 19.4 -> 20.3 mm
- removed copper zone on F.Cu, net +5V

Commit message: rerouted several PCBs
Parts:
- removed REF** (x2): MountingHole_3.2mm_M3, MountingHole:MountingHole_3.2mm_M3

Commit message: added dcc sniffer, conversion to kicad 6
Other:
- net class Default removed
